Commit message: replace gen3 base_link to kortex_base_link

File: kortex_description/arms/gen3/7dof/urdf/gen3_macro.xacro (robot description, xacro)
@@ -4,5 +4,5 @@
   <xacro:property name="last_arm_link" value="end_effector_link"/>
   <xacro:macro name="load_arm" params="parent:='' dof vision *origin">
-      <link name="base_link">
+      <link name="kortex_base_link">
         <inertial>
           <origin xyz="-0.000648 -0.000166 0.084487" rpy="0 0 0" />
@@ -53,5 +53,5 @@
       <origin xyz="0 0 0.15643" rpy="3.1416 2.7629E-18 -4.9305E-36" />
       <parent
-        link="base_link" />
+        link="kortex_base_link" />
       <child
         link="shoulder_link" />
